File: Hardware Design Kicad 9.0/IAQ_AIQALLINone/IAQ_AIQALLINone.kicad_sch (KiCad schematic)
At the start: 6 parts, among them IC1 ENS160-BGLT, IC2 SGP41-D-R4, U1 RASPBERRY_PI_4B_4GB, U2 RASPBERRY_PI_PICO_W, U3 BME688

Commit message: update
141619032026
Parts:
- U2: footprint RASPBERRY_PI_PICO_W:MODULE_RASPBERRY_PI_PICO_W -> Module:RaspberryPi_Pico_W_SMD_HandSolder
Changed lines of the file:
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@@
 			)
 		)
-		(property "Footprint" "RASPBERRY_PI_PICO_W:MODULE_RASPBERRY_PI_PICO_W"
+		(property "Footprint" "Module:RaspberryPi_Pico_W_SMD_HandSolder"
 			(at 825.5 193.04 0)
 			(effects
